Commit message: [Upd] Working config

File: velodyne_description/urdf/lio-sam-test-1.urdf.xacro (robot description, xacro)
@@ -5,7 +5,11 @@
   <xacro:arg name="organize_cloud" default="false"/>
   <xacro:property name="organize_cloud" value="$(arg organize_cloud)" />
+  <xacro:include filename="common_properties.xacro"/>
+  <xacro:include filename="mobile_base.xacro"/>
+  <xacro:include filename="mobile_base_gazebo.xacro"/>
+  <xacro:include filename="camera.xacro"/>
+  <!-- <xacro:include filename="lidar.xacro"/> -->
   <!-- Base Footprint -->
-  <link name="base_footprint" />
-  <!-- Base Link -->
+  <!-- <link name="base_footprint" />
   <joint name="footprint" type="fixed" >
    <parent link="base_footprint" />
@@ -31,52 +35,8 @@
                izz="3.0" />
     </inertial>
-  </link>
-  <joint name="base_imu_joint" type="fixed">
-    <parent link="base_link" />
-    <child link="imu_link" />
-    <origin xyz="0 0 0.44085" rpy="0 0 0" />
-  </joint>
-  <link name="imu_link">
-    <visual>
-      <geometry>
-        <box size="0.1 0.1 0.03" />
-      </geometry>
-      <material name="grey" />
-    </visual>
-    <collision>
-      <origin rpy="0 0 0" xyz="0 0 0.44085"/>
-      <geometry>
-        <box size="0.1 0.1 0.03" />
-      </geometry>
-      <material name="grey"/>
-    </collision>
-    <inertial>
-      <origin xyz="0 0 0.44085" rpy="0 0 0"/>
-      <mass value="1.0" />
-      <inertia ixx="0.3" ixy="0" ixz="0"
-               iyy="0.3" iyz="0"
-               izz="0.3"/>
-    </inertial>
-  </link>
-  <gazebo reference="imu_link">
-      <gravity>true</gravity>
-      <sensor name="imu_sensor" type="imu">
-        <always_on>true</always_on>
-        <update_rate>100</update_rate>
-        <visualize>true</visualize>
-        <topic>/imu/data</topic>
-        <plugin filename="libgazebo_ros_imu_sensor.so" name="imu_plugin">
-          <topicName>/imu/data</topicName>
-          <bodyName>imu_link</bodyName>
-          <updateRateHZ>100.0</updateRateHZ>
-          <gaussianNoise>0.000000001</gaussianNoise>
-          <xyzOffset>0 0 0</xyzOffset>
-          <rpyOffset>0 0 0</rpyOffset>
-          <frameName>imu_link</frameName>
-          <initialOrientationAsReference>false</initialOrientationAsReference>
-        </plugin>
-        <pose>0 0 0 0 0 0</pose>
-      </sensor>
-    </gazebo>
+  </link> -->
+  <!-- IMU Link -->
+  <xacro:include filename="imu-sensor.xacro"/>
+  <!-- Lidars -->
   <xacro:include filename="$(find velodyne_description)/urdf/VLP-16.urdf.xacro"/>
   <xacro:VLP-16 parent="base_link" name="velodyne" topic="/os_cloud_node/points" organize_cloud="${organize_cloud}" hz="10" samples="440" gpu="${gpu}">
